File: Hardware/Echoes_of_Termina/Echoes_of_Termina.kicad_pcb (KiCad board)
At the start: 2 copper layers, 99 x 59.5 mm, 82 parts, among them J1 USB_C_Receptacle_USB2.0_8P, J2 Conn_01x03_Socket, J3 Conn_01x02_Socket, J4 Conn_01x02_Socket, Q1 PMOS, Q2 2N7002K, Q3 PMOS, U1 TP4056, U2 AP2112K-3.3, U3 ESP32-WROOM-32, U4 MAX98357A, U5 MAX98357A, U6 INMP441

Commit message: 0.7
Parts:
- C1, C12, C13, C14, C15, C16, C17, C18, C2, C3, C4, C5, C6, C8: footprint Capacitor_SMD:C_0805_2012Metric -> Capacitor_SMD:C_0805_2012Metric_Pad1.18x1.45mm_HandSolder
- L1: footprint Inductor_SMD:L_0805_2012Metric -> Inductor_SMD:L_0805_2012Metric_Pad1.05x1.20mm_HandSolder
- R10, R16, R17, R18, R19, R20, R21, R22, R23, R24, R25, R3, R4, R6, R7, R9: footprint Resistor_SMD:R_0805_2012Metric -> Resistor_SMD:R_0805_2012Metric_Pad1.20x1.40mm_HandSolder
- R11: value 330R -> 330; footprint Resistor_SMD:R_0805_2012Metric -> Resistor_SMD:R_0805_2012Metric_Pad1.20x1.40mm_HandSolder
- U3: value ESP32-WROOM-32 -> ESP32-WROOM-32U-N8
- moved D4 0.35 mm to (190.7, 122.9)
- moved R10 0.33 mm to (203.9, 119.7)
- moved R17 0.23 mm to (200.4, 121.7)
Routing:
- net Button_GPIO: track 89.8 -> 79.1 mm
- net GND: track 5.09 -> 5.21 mm, vias 88 -> 91
