File: Hardware/Marajoara_V3/Marajoara_V3.kicad_pcb (KiCad board)
At the start: 2 copper layers, 222.6 x 162.8 mm, 95 parts, among them J1 USB_C_Receptacle_USB2.0_8P, J3 Conn_01x02_Socket, J4 Conn_01x02_Socket, Q1 PMOS, Q2 2N7002K, Q3 PMOS, U1 TP4056, U2 AP2112K-3.3, U3 ESP32-WROOM-32-N8R2, U4 MAX98357A, U5 MAX98357A, U6 INMP441

Commit message: Update Setembro
Parts:
- removed the BT3 at (184.6, 134.7)
- removed the C8 at (187.7, 140.1)
- removed D2: LED_BLUE, LED_SMD:LED_0805_2012Metric_Pad1.15x1.40mm_HandSolder
- removed D8, D9: SS14, Diode_SMD:D_SMA
- removed the R10 at (167.4, 135.9)
- removed the R20 at (161.9, 152.4)
- removed the R25 at (172.8, 123.9)
- removed the R5 at (182.4, 123.5)
- removed the R6 at (187.2, 115.3)
- removed the R7 at (184.9, 115.3)
- removed the R8 at (184.0, 140.1)
- removed the R9 at (180.1, 140.1)
- removed the U2 at (52.3, 108.0)
- added BATT2: Conn_01x02_Socket, Connector_Molex:Molex_KK-254_AE-6410-02A_1x02_P2.54mm_Vertical, F.Cu at (273.4, 145.9)
- added BT4: SW_Push, Button_Switch_SMD:SW_SPST_PTS647_Sx38, F.Cu at (166.4, 184.1)
- added C15: 220uF, Aleoexpress:Cap_polymer, F.Cu at (247.2, 109.5)
- added C18: 100n, Capacitor_SMD:C_0805_2012Metric_Pad1.18x1.45mm_HandSolder, F.Cu at (271.4, 58.4)
- added C19: 100n, Capacitor_SMD:C_0805_2012Metric_Pad1.18x1.45mm_HandSolder, F.Cu at (307.4, 127.6)
- added C20: 100n, Capacitor_SMD:C_0805_2012Metric_Pad1.18x1.45mm_HandSolder, F.Cu at (294.7, 155.0)
- added C21: 100n, Capacitor_SMD:C_0805_2012Metric_Pad1.18x1.45mm_HandSolder, F.Cu at (270.3, 182.9)
- added C22: 100n, Capacitor_SMD:C_0805_2012Metric_Pad1.18x1.45mm_HandSolder, F.Cu at (238.8, 206.3)
- added C23: 100n, Capacitor_SMD:C_0805_2012Metric_Pad1.18x1.45mm_HandSolder, F.Cu at (166.6, 205.6)
- added C24: 100n, Capacitor_SMD:C_0805_2012Metric_Pad1.18x1.45mm_HandSolder, F.Cu at (135.1, 181.6)
- added C25: 100n, Capacitor_SMD:C_0805_2012Metric_Pad1.18x1.45mm_HandSolder, F.Cu at (114.0, 155.5)
- added C26: 100n, Capacitor_SMD:C_0805_2012Metric_Pad1.18x1.45mm_HandSolder, F.Cu at (99.5, 125.0)
- added C27: 100n, Capacitor_SMD:C_0805_2012Metric_Pad1.18x1.45mm_HandSolder, F.Cu at (135.8, 58.4)
- added C28: 100n, Capacitor_SMD:C_0805_2012Metric_Pad1.18x1.45mm_HandSolder, F.Cu at (153.6, 185.2)
- added C9: 10u, Capacitor_SMD:C_0805_2012Metric_Pad1.18x1.45mm_HandSolder, F.Cu at (183.0, 182.3)
- added D5: SS14, Diode_SMD:D_SMA, F.Cu at (171.9, 156.4)
- added H3: MountingHole, MountingHole:MountingHole_3.2mm_M3, F.Cu at (265.6, 172.5)
- added H4: MountingHole, MountingHole:MountingHole_3.2mm_M3, F.Cu at (140.6, 172.5)
- added J2: USB_C_Receptacle_USB2.0_8P, Aleoexpress:USB-C-SMD_GT-USB-7101A, F.Cu at (184.6, 164.1)
- added Q4: PMOS, Package_TO_SOT_SMD:SOT-23_Handsoldering, F.Cu at (167.9, 157.1)
- added R15: 2.2k, Resistor_SMD:R_0805_2012Metric_Pad1.20x1.40mm_HandSolder, F.Cu at (188.2, 174.4)
- added R18: 10k, Resistor_SMD:R_0805_2012Metric_Pad1.20x1.40mm_HandSolder, F.Cu at (161.2, 184.7)
- added R19: 100k, Resistor_SMD:R_0805_2012Metric_Pad1.20x1.40mm_HandSolder, F.Cu at (151.1, 187.2)
- added R22: 100k, Resistor_SMD:R_0805_2012Metric, F.Cu at (166.9, 162.2)
- added R28: 100k, Resistor_SMD:R_0805_2012Metric_Pad1.20x1.40mm_HandSolder, F.Cu at (163.7, 179.1)
- added R29: 330, Resistor_SMD:R_0805_2012Metric_Pad1.20x1.40mm_HandSolder, F.Cu at (149.8, 172.7)
- added R3: 5.1k, Resistor_SMD:R_0805_2012Metric_Pad1.20x1.40mm_HandSolder, F.Cu at (177.2, 165.2)
- added R30: 10k, Resistor_SMD:R_0805_2012Metric_Pad1.20x1.40mm_HandSolder, F.Cu at (155.5, 177.3)
- added R31: 10k, Resistor_SMD:R_0805_2012Metric_Pad1.20x1.40mm_HandSolder, F.Cu at (158.2, 83.4)
- added R32: 220k, Resistor_SMD:R_0805_2012Metric_Pad1.20x1.40mm_HandSolder, F.Cu at (249.3, 96.6)
- added U6: TP4056, Aleoexpress:ESOP-8_L4.9-W3.9-P1.27-LS6.0-BL-EP, F.Cu at (181.1, 177.9)
- added U7: MAX98357AETE+T, Aleoexpress:TQFN-16_L3.0-W3.0-P0.50-BL-EP1.5, F.Cu at (155.7, 87.5)
- added U8: MAX98357AETE+T, Aleoexpress:TQFN-16_L3.0-W3.0-P0.50-BL-EP1.5, F.Cu at (251.9, 92.5)
- BOTTOM1, EYE1, EYE2, MID1, PORT1, PORT2, TOP1: footprint Connector_Hirose:Hirose_DF13C_CL535-0404-8-51_1x04-1MP_P1.25mm_Vertical -> Aleoexpress:Hirose_DF13C_CL535-0404-8-51_1x04-1MP_P1.25mm_Vertical
- C4: value 10u -> 100n
- D3: value LED_RED -> LED_BLUE
- D4: value SS14 -> LED_RED; footprint Diode_SMD:D_SMA -> LED_SMD:LED_0805_2012Metric_Pad1.15x1.40mm_HandSolder
- J1: value USB_C_Receptacle_USB2.0_8P -> Conn_01x02_Socket; footprint Aleoexpress:USB-C-SMD_GT-USB-7101A -> Connector_Molex:Molex_KK-254_AE-6410-02A_1x02_P2.54mm_Vertical
- R1: value 2.2k -> 100k; footprint Resistor_SMD:R_0805_2012Metric -> Resistor_SMD:R_0805_2012Metric_Pad1.20x1.40mm_HandSolder
- R16: value 330 -> 220mR 1W 1%; footprint Resistor_SMD:R_0805_2012Metric_Pad1.20x1.40mm_HandSolder -> Resistor_SMD:R_1206_3216Metric_Pad1.30x1.75mm_HandSolder
- R17: value 10k -> 2.2k
- R2: value 220mR 1W 1% -> 5.1k; footprint Resistor_SMD:R_1206_3216Metric_Pad1.30x1.75mm_HandSolder -> Resistor_SMD:R_0805_2012Metric_Pad1.20x1.40mm_HandSolder
- R21: renamed from R19; value 100k -> 220k
- R27: renamed from R12; footprint Resistor_SMD:R_0805_2012Metric -> Resistor_SMD:R_0805_2012Metric_Pad1.20x1.40mm_HandSolder
- R6: renamed from R11; value 330 -> 2.2k
- R7: renamed from R26; footprint Resistor_SMD:R_0805_2012Metric -> Resistor_SMD:R_0805_2012Metric_Pad1.20x1.40mm_HandSolder
- R8: renamed from R27; footprint Resistor_SMD:R_0805_2012Metric -> Resistor_SMD:R_0805_2012Metric_Pad1.20x1.40mm_HandSolder
- U1: value TP4056 -> AP2112K-3.3; footprint Aleoexpress:ESOP-8_L4.9-W3.9-P1.27-LS6.0-BL-EP -> Package_TO_SOT_SMD:SOT-23-5
- moved C6 144.1 mm to (186.3, 107.8), turned to 0 degrees
- moved BT2 143.7 mm to (181.5, 103.6), turned to 0 degrees
- moved C4 131.7 mm to (175.5, 146.2), turned to 0 degrees
- moved H2 115.5 mm to (265.6, 107.5)
- moved D4 113.8 mm to (188.3, 176.8)
- moved L1 113.3 mm to (189.7, 118.1)
- moved R5 112.9 mm to (191.8, 118.3)
- moved C2 112.7 mm to (189.7, 112.9)
- moved C3 112.7 mm to (192.2, 112.9)
- moved D1 110.7 mm to (187.1, 112.8), turned to -90 degrees
- moved R6 110.3 mm to (187.1, 118.3), turned to -90 degrees
- moved U2 107.0 mm to (204.0, 121.0)
- moved BT1 105.1 mm to (217.2, 131.8), turned to -90 degrees
- moved EYE1 102.1 mm to (155.1, 129.4), turned to -90 degrees
- moved C13 100.5 mm to (163.0, 76.9)
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- renumbered BT4 to BT3, C17 to C10, C12 to C11, C7 to C12, C15 to C16, C16 to C17, C5 to C2, C6 to C3, C2 to C5, C3 to C6, C18 to C7, C19 to C8, D5 to D1, JP3 to JP1, JP1 to JP2, JP2 to JP3, R29 to R10, R30 to R11, R31 to R12, R32 to R13, R33 to R14, R18 to R20, R22 to R23, R23 to R25, R24 to R26, R3 to R4, R4 to R5, R28 to R9, U3 to U2, U6 to U3
Connections:
- net Net-(JP2-C) renamed GAIN_R
- net Net-(S10-DOUT) renamed /Top1_IN
- BOTTOM1 pad 1: Net-(BOTTOM1-Pin_1) -> /Eye1_OUT
- BOTTOM1 pad 3: V_REG -> VCC
- BOTTOM1 pad 4: unconnected-(BOTTOM1-Pin_4-Pad4) -> Net-(BOTTOM1-Pin_4)
- C1 pad 1: +BATT -> +3.3V
- C12 pad 1: V_SPK -> VCC
- C13 pad 1: V_SPK -> VCC
- C14 pad 2: V_SPK -> VCC
- C16 pad 1: V_SPK -> VCC
- C17 pad 2: V_SPK -> VCC
- C4 pad 1: +3.3V -> Net-(U1-EN)
- D1 pad 2: Net-(D5-A) -> Net-(D1-A)
- D3 pad 2: Net-(D2-A) -> Net-(D3-A)
- D4 pad 2: V_REG -> Net-(D3-A)
- EYE1 pad 1: Net-(EYE1-Pin_1) -> /Top1_OUT
- EYE1 pad 3: V_REG -> VCC
- EYE1 pad 4: Net-(EYE1-Pin_4) -> /Eye1_OUT
- EYE2 pad 1: Net-(EYE1-Pin_4) -> Net-(EYE2-Pin_1)
- EYE2 pad 3: V_REG -> VCC
- EYE2 pad 4: Net-(EYE2-Pin_4) -> unconnected-(EYE2-Pin_4-Pad4)
- JP2 pad 2: Net-(JP1-C) (its old number) -> GAIN_L
- JP2 pad 3: V_SPK -> VCC
- JP3 pad 3: V_SPK -> VCC
- MID1 pad 1: Net-(MID1-Pin_1) -> Net-(BOTTOM1-Pin_4)
- MID1 pad 3: V_REG -> VCC
- MID1 pad 4: Net-(BOTTOM1-Pin_1) -> Net-(EYE2-Pin_1)
- Q3 pad 2: V_SPK -> Net-(Q3-S)
- R1 pad 1: +5V -> VCC
- R1 pad 2: Net-(D2-A) -> Net-(U1-EN)
- R16 pad 1: latch_enable -> +5V
- R16 pad 2: Net-(D7-A) -> Net-(U6-CE)
- R17 pad 1: Net-(D6-K) -> GND
- R17 pad 2: GND -> Net-(U6-PROG)
- R2 pad 1: +5V -> GND
- R2 pad 2: Net-(U1-VCC) -> Net-(J2-CC2)
- R20 pad 2: V_REG -> VCC
- R21 pad 1: Net-(R19-Pad1) -> ADC1_0
- R25 pad 1: V_SPK -> VCC
- R26 pad 1: V_SPK -> VCC
- R27 pad 1: Majora_out -> Strip_out
- R27 pad 2: Net-(EYE1-Pin_1) -> Net-(S1-DIN)
- R6 pad 1: +3.3V -> Net-(D1-A)
- R6 pad 2: Net-(D5-A) -> +3.3V
- S1 pad 1: Net-(EYE2-Pin_4) -> Net-(S1-DIN)
- S1 pad 3: V_REG -> VCC
- S10 pad 3: V_REG -> VCC
- S2 pad 3: V_REG -> VCC
- S3 pad 3: V_REG -> VCC
- S4 pad 3: V_REG -> VCC
- S5 pad 3: V_REG -> VCC
- S6 pad 3: V_REG -> VCC
- S7 pad 3: V_REG -> VCC
- S8 pad 3: V_REG -> VCC
- S9 pad 3: V_REG -> VCC
- TOP1 pad 3: V_REG -> VCC
- TOP1 pad 4: Net-(MID1-Pin_1) -> /Top1_OUT
- U1 pad 1: GND -> VCC
- U1 pad 2: Net-(U1-PROG) -> GND
- U1 pad 3: GND -> Net-(U1-EN)
- U1 pad 4: Net-(U1-VCC) -> unconnected-(U1-NC-Pad4)
- U1 pad 5: +BATT -> +3.3V
- U2 pad 37: latch_enable -> Strip_out
- U2 pad 8: Strip_out -> latch_enable
- U4 pad 4: Net-(JP1-C) (its old number) -> GAIN_L
- U4 pad 7: V_SPK -> VCC
- U4 pad 8: Net-(J3-Pin_1) -> unconnected-(U4-Out+-Pad8)
- U4 pad 9: Net-(J3-Pin_2) -> unconnected-(U4-Out--Pad9)
- U5 pad 7: V_SPK -> VCC
- U5 pad 8: Net-(J4-Pin_1) -> unconnected-(U5-Out+-Pad8)
- U5 pad 9: Net-(J4-Pin_2) -> unconnected-(U5-Out--Pad9)
Routing:
- net VCC: track 0.00 -> 915.4 mm
- net +BATT: track 42.6 -> 214.9 mm
- net I2S_DOUT: track 0.00 -> 167.2 mm, vias 0 -> 1
- net I2S_BCLK: track 0.00 -> 165.7 mm, vias 0 -> 1
- net I2S_LRC: track 14.4 -> 163.8 mm, vias 0 -> 1
- net /Eye1_OUT: track 0.00 -> 123.1 mm
- net +3.3V: track 85.7 -> 178.6 mm, vias 1 -> 0
- net Net-(S10-DIN): track 0.00 -> 88.9 mm
- net Net-(S1-DOUT): track 0.00 -> 88.0 mm
- net Net-(S5-DOUT): track 0.00 -> 87.7 mm
- net Button_GPIO: track 54.2 -> 137.7 mm, vias 5 -> 1
- net Net-(EYE2-Pin_1): track 0.00 -> 83.3 mm
- net Net-(S1-DIN): track 0.00 -> 75.1 mm
- net /Top1_IN: track 0.00 -> 56.9 mm
- net /Top1_OUT: track 0.00 -> 55.0 mm
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Other:
- board size 222.6 x 162.8 mm -> 230.7 x 176.5 mm
- board text removed: "Botão + Power on"
- board text removed: "Carregador 4.2V 500mA"
- board text removed: "Cartão MicroSD SDMMC"
- board text removed: "I2C"
- board text removed: "Microfone INMP441"
- board text removed: "Serial"

Commit message: Hardware update
hardware: Marajoara V3 routing refresh, Echoes case/3D — KiCad + production outputs + Case/, Speaker_40mm_Case/
Parts:
- added C29: 220uF, Aleoexpress:Cap_polymer, F.Cu at (245.4, 192.8)
- added D9: LED_GREEN, LED_SMD:LED_0805_2012Metric_Pad1.15x1.40mm_HandSolder, F.Cu at (179.7, 146.9)
- added J5: Conn_01x03_Socket, TerminalBlock:TerminalBlock_Xinya_XY308-2.54-3P_1x03_P2.54mm_Horizontal, F.Cu at (236.0, 192.8)
- added R24: 10k, Resistor_SMD:R_0805_2012Metric_Pad1.20x1.40mm_HandSolder, F.Cu at (216.4, 126.6)
- added R33: 0R, Resistor_SMD:R_0805_2012Metric_Pad1.20x1.40mm_HandSolder, B.Cu at (204.1, 151.8)
- added R34: 330, Resistor_SMD:R_0805_2012Metric_Pad1.20x1.40mm_HandSolder, F.Cu at (226.2, 147.0)
- added R36: 2.2k, Resistor_SMD:R_0805_2012Metric_Pad1.20x1.40mm_HandSolder, F.Cu at (179.7, 151.0)
- D5: value SS14 -> SS34; footprint Diode_SMD:D_SMA -> Diode_SMD:D_SMC_Handsoldering
- R22: value 100k -> 10k; footprint Resistor_SMD:R_0805_2012Metric -> Resistor_SMD:R_0805_2012Metric_Pad1.20x1.40mm_HandSolder
- U2: footprint RF_Module:ESP32-WROOM-32U -> PCM_Espressif:ESP32-WROOM-32UE
- moved Q3 7.36 mm to (169.4, 171.5)
- moved R22 6.83 mm to (160.4, 164.3), turned to 180 degrees
- moved Q4 6.80 mm to (164.3, 162.9)
- moved D5 1.72 mm to (170.5, 157.4)
Connections:
- net MIC_SCK renamed I2S_MIC_BCLK
- net MIC_SD renamed I2S_MIC_D
- net MIC_WS renamed I2S_MIC_WS
- R27 pad 1: Strip_out -> Mask_out
- U2 pad 12: SD_D2 -> I2S_SPK_BCLK
- U2 pad 16: SD_D3 -> I2S_SPK_D
- U2 pad 27: I2S_DOUT -> Net-(U2-IO16)
- U2 pad 28: I2S_BCLK -> unconnected-(U2-IO17-Pad28)
- U2 pad 37: Strip_out -> Mask_out
- U2 pad 9: unconnected-(U2-IO33-Pad9) -> Strip_out
- U4 pad 2: I2S_BCLK -> I2S_SPK_BCLK
- U4 pad 3: I2S_DOUT -> I2S_SPK_D
- U5 pad 2: I2S_BCLK -> I2S_SPK_BCLK
- U5 pad 3: I2S_DOUT -> I2S_SPK_D
- U7 pad 1: I2S_DOUT -> I2S_SPK_D
- U7 pad 16: I2S_BCLK -> I2S_SPK_BCLK
- U8 pad 1: I2S_DOUT -> I2S_SPK_D
- U8 pad 16: I2S_BCLK -> I2S_SPK_BCLK
Routing:
- net I2S_SPK_BCLK: track 0.00 -> 168.1 mm, vias 0 -> 1
- net I2S_DOUT: track 167.2 -> 0.00 mm, vias 1 -> 0
- net I2S_SPK_D: track 0.00 -> 166.9 mm, vias 0 -> 1
- net I2S_BCLK: track 165.7 -> 0.00 mm, vias 1 -> 0
- net Net-(J5-Pin_2): track 0.00 -> 47.9 mm, vias 0 -> 2
- net Strip_out: track 18.0 -> 49.9 mm, vias 0 -> 2
- net VCC: track 915.4 -> 936.6 mm
- net +3.3V: track 178.6 -> 197.6 mm, vias 0 -> 2
- net Mask_out: track 0.00 -> 18.0 mm
- net SD_D3: track 30.2 -> 12.5 mm, vias 2 -> 0
- net SD_D2: track 24.9 -> 13.3 mm
- net +5V: track 37.7 -> 47.3 mm
- net V_REG: track 13.9 -> 6.07 mm
- net I2S_MIC_D: track 30.9 -> 35.4 mm
- net Net-(U2-IO16): track 0.00 -> 2.67 mm
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