File: Hardware/Marajoara_V3/Marajoara_V3.kicad_sch (KiCad schematic)
At the start: 98 parts, among them J1 USB_C_Receptacle_USB2.0_8P, J3 Conn_01x02_Socket, J4 Conn_01x02_Socket, Q1 PMOS, Q2 2N7002K, Q3 PMOS, U1 TP4056, U2 AP2112K-3.3, U3 ESP32-WROOM-32-N8R2, U4 MAX98357A, U5 MAX98357A, U6 INMP441

Commit message: Update Setembro
Parts:
- removed D9: SS14, Diode_SMD:D_SMA, symbol Diode:SS14
- removed R19, R20, R25: 100k, Resistor_SMD:R_0805_2012Metric_Pad1.20x1.40mm_HandSolder, symbol Device:R
- removed R8: 2.2k, Resistor_SMD:R_0805_2012Metric_Pad1.20x1.40mm_HandSolder, symbol Device:R
- added BATT2, J1: Conn_01x02_Socket, Connector_Molex:Molex_KK-254_AE-6410-02A_1x02_P2.54mm_Vertical, symbol Connector:Conn_01x02_Socket
- added C15: 220uF, Aleoexpress:Cap_polymer, symbol Device:C_Polarized
- added C18, C19, C20, C21, C22, C23, C24, C25, C26, C27: 100n, Capacitor_SMD:C_0805_2012Metric_Pad1.18x1.45mm_HandSolder, symbol Device:C
- added D5: SS14, Diode_SMD:D_SMA, symbol Diode:SS14
- added Q4: PMOS, Package_TO_SOT_SMD:SOT-23_Handsoldering, symbol Simulation_SPICE:PMOS
- added R18, R22, R31: 10k, Resistor_SMD:R_0805_2012Metric_Pad1.20x1.40mm_HandSolder, symbol Device:R
- added R21, R32: 220k, Resistor_SMD:R_0805_2012Metric_Pad1.20x1.40mm_HandSolder, symbol Device:R
- added U7, U8: MAX98357AETE+T, Aleoexpress:TQFN-16_L3.0-W3.0-P0.50-BL-EP1.5, symbol ALeoExpress:MAX98357AETE+T
- BOTTOM1, EYE1, EYE2, MID1, PORT1, PORT2, TOP1: footprint Connector_Hirose:Hirose_DF13C_CL535-0404-8-51_1x04-1MP_P1.25mm_Vertical -> Aleoexpress:Hirose_DF13C_CL535-0404-8-51_1x04-1MP_P1.25mm_Vertical
- D2: renamed from D8; now not fitted; now left out of the parts list
- U4, U5: now left out of the parts list
- renumbered BT4 to BT3, BT3 to BT4, C4 to C1, C17 to C10, C12 to C11, C7 to C12, C15 to C16, C16 to C17, C5 to C2, C8 to C28, C6 to C3, C9 to C4, C2 to C5, C3 to C6, C18 to C7, C19 to C8, C1 to C9, D5 to D1, D2 to D3, D3 to D4, J1 to J2, JP3 to JP1, JP1 to JP2, JP2 to JP3, R13 to R1, R29 to R10, R30 to R11, R31 to R12, R32 to R13, R33 to R14, R1 to R15, R2 to R16, R5 to R17, R9 to R19, R6 to R2, R18 to R20, R22 to R23, R23 to R25, R24 to R26, R12 to R27, R10 to R28, R16 to R29, R7 to R3, R17 to R30, R3 to R4, R4 to R5, R11 to R6, R26 to R7, R27 to R8, R28 to R9, U2 to U1, U3 to U2, U6 to U3, U1 to U6
Connections:
- net Majora_out is gone; now on net Strip_out: R27.1
- net +5V: now also D5.2 (A), J1.1 (Pin_1), Q4.1 (G), R22.1; no longer R15.1, U6.8 (CE)
- net +BATT: now also BATT2.1 (Pin_1)
- net ADC1_0: now also R21.1
- net Button_GPIO: now also R19.2, R18.1
- net GND: now also BATT2.2 (Pin_2), C15.2, C18.2, C19.2, C20.2, C21.2, C22.2, C23.2, C24.2, C25.2, C26.2, C27.2, J1.2 (Pin_2), R22.2, U7.11 (GND), U7.15 (GND), U7.17 (EP), U7.3 (GND), U8.11 (GND), U8.15 (GND), U8.17 (EP), U8.3 (GND)
- net I2S_BCLK: now also U7.16 (BCLK), U8.16 (BCLK)
- net I2S_DOUT: now also U7.1 (DIN), U8.1 (DIN)
- net I2S_LRC: now also U7.14 (LRCLK), U8.14 (LRCLK)
- net Strip_out: now also U2.37 (IO23); no longer U2.8 (IO32)
- net V_REG: no longer BOTTOM1.3 (Pin_3), EYE1.3 (Pin_3), EYE2.3 (Pin_3), MID1.3 (Pin_3), R1.1, R20.2, S1.3 (VDD), S10.3 (VDD), S2.3 (VDD), S3.3 (VDD), S4.3 (VDD), S5.3 (VDD), S6.3 (VDD), S7.3 (VDD), S8.3 (VDD), S9.3 (VDD), TOP1.3 (Pin_3), U1.1 (VIN)
- net latch_enable: now also U2.8 (IO32); no longer U2.37 (IO23)
- net at R16.2, U6.4 (VCC): now also R15.2, U6.8 (CE)
- net at S1.1 (DIN): now also R27.2; no longer EYE2.4 (Pin_4)
- net at MID1.4 (Pin_4): now also EYE2.1 (Pin_1); no longer BOTTOM1.1 (Pin_1)
- net at BOTTOM1.4 (Pin_4): now also MID1.1 (Pin_1)
- net at J3.1 (Pin_1): now also U7.9 (OUTP); no longer U4.8 (Out+)
- net at J3.2 (Pin_2): now also U7.10 (OUTN); no longer U4.9 (Out-)
- net at BT4.2: now also R18.2; no longer R19.2
- net GAIN_R: now reaches JP3.2 (C), U5.4 (GAIN)
- net GAIN_R: now also U8.2 (GAIN_SLOT)
- net at U5.8 (Out+): no longer J4.1 (Pin_1)
- net at U5.9 (Out-): no longer J4.2 (Pin_2)
- net Eye1_OUT: now reaches EYE1.4 (Pin_4)
- net Eye1_OUT: now also BOTTOM1.1 (Pin_1); no longer EYE2.1 (Pin_1)
- net at D3.2 (A), D4.2 (A): now also R15.1; no longer R15.2
- net Top1_OUT: now reaches TOP1.4 (Pin_4)
- net Top1_OUT: now also EYE1.1 (Pin_1); no longer MID1.1 (Pin_1)
- net Top1_IN: now reaches S10.4 (DOUT), TOP1.1 (Pin_1)
- net GAIN_L: now reaches JP2.2 (C), U4.4 (GAIN)
- net GAIN_L: now also U7.2 (GAIN_SLOT)
- net at R20.1: now also R21.2
- net V_SPK renamed VCC
- net VCC: now also BOTTOM1.3 (Pin_3), EYE1.3 (Pin_3), EYE2.3 (Pin_3), MID1.3 (Pin_3), R1.1, R20.2, S1.3 (VDD), S10.3 (VDD), S2.3 (VDD), S3.3 (VDD), S4.3 (VDD), S5.3 (VDD), S6.3 (VDD), S7.3 (VDD), S8.3 (VDD), S9.3 (VDD), TOP1.3 (Pin_3), U1.1 (VIN), C15.1, C18.1, C19.1, C20.1, C21.1, C22.1, C23.1, C24.1, C25.1, C26.1, C27.1, D5.1 (K), Q4.3 (D), R31.1, R32.2, U7.7 (VDD), U7.8 (VDD), U8.7 (VDD), U8.8 (VDD); no longer Q3.2 (S)
- new net: R31.2, U7.4 (~{SD_MODE})
- new net: Q3.2 (S), Q4.2 (S)
- new net: R32.1, U8.4 (~{SD_MODE})
- new net: J4.2 (Pin_2), U8.10 (OUTN)
- new net: J4.1 (Pin_1), U8.9 (OUTP)
- no-connect marks 11 -> 15
Other:
- note added: "Open G=9 VDD G=6 100k G=3"
- note added: "PMOS blocks battery drain in case of VCC present"
- note added: "Spikes decoupling caps"
- note added: "Voltage source constrainer"
- note removed: "Open G=9 100k G=6 0R G=3"
- moved on the sheet: BATT1, BOTTOM1, C13, C14, C16, C17, C28, C9, D3, D4, D7, EYE1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

Commit message: Hardware update
hardware: Marajoara V3 routing refresh, Echoes case/3D — KiCad + production outputs + Case/, Speaker_40mm_Case/
Parts:
- removed D5: SS14, Diode_SMD:D_SMA, symbol Diode:SS14
- added C29: 220uF, Aleoexpress:Cap_polymer, symbol Device:C_Polarized
- added D5: SS34, Diode_SMD:D_SMC_Handsoldering, symbol Diode:SS34
- added D9: LED_GREEN, LED_SMD:LED_0805_2012Metric_Pad1.15x1.40mm_HandSolder, symbol Device:LED
- added J5: Conn_01x03_Socket, TerminalBlock:TerminalBlock_Xinya_XY308-2.54-3P_1x03_P2.54mm_Horizontal, symbol Connector:Conn_01x03_Socket
- added R24: 10k, Resistor_SMD:R_0805_2012Metric_Pad1.20x1.40mm_HandSolder, symbol Device:R
- added R33: 0R, Resistor_SMD:R_0805_2012Metric_Pad1.20x1.40mm_HandSolder, symbol Device:R
- added R34: 330, Resistor_SMD:R_0805_2012Metric_Pad1.20x1.40mm_HandSolder, symbol Device:R
- added R36: 2.2k, Resistor_SMD:R_0805_2012Metric_Pad1.20x1.40mm_HandSolder, symbol Device:R
- TF1: footprint ALeoExpress:TF-SMD_TF-CARD-XG8P-H1.5 -> Aleoexpress:TF-SMD_TF-CARD-XG8P-H1.5
- U2: footprint RF_Module:ESP32-WROOM-32-N8R2 -> PCM_Espressif:ESP32-WROOM-32UE
Connections:
- net +3.3V: now also R24.1
- net +5V: now also D5.2 (A)
- net GND: now also C29.2, D9.1 (K), J5.3 (Pin_3)
- net SD_D2: no longer U2.12 (IO27)
- net SD_D3: no longer U2.16 (IO13)
- net Strip_out: now also U2.9 (IO33), R34.1; no longer R27.1, U2.37 (IO23)
- net VCC: now also C29.1, D5.1 (K), J5.1 (Pin_1), R36.2
- net I2S_BCLK renamed I2S_SPK_BCLK
- net I2S_SPK_BCLK: now also U2.12 (IO27); no longer U2.28 (IO17)
- net I2S_DOUT renamed I2S_SPK_D
- net I2S_SPK_D: now also U2.16 (IO13); no longer U2.27 (IO16)
- net MIC_SCK renamed I2S_MIC_BCLK
- net MIC_SD renamed I2S_MIC_D
- net MIC_WS renamed I2S_MIC_WS
- new net: J5.2 (Pin_2), R34.2
- new net: R24.2, U2.27 (IO16)
- new net: D9.2 (A), R36.1
- new net Mask_out: R27.1, U2.37 (IO23)
- no-connect marks 15 -> 16
Other:
- note added: "PSRAM Pins"
- note added: "Strip Output"
- moved on the sheet: BT3, D1, JP1, R6, U4, U5
