File: Hardware/PCBs/Marajoara_V3/Marajoara_V3.kicad_pcb (KiCad board)
At the start: 2 copper layers, 230.7 x 176.5 mm, 121 parts, among them J1 Conn_01x02_Socket, J2 USB_C_Receptacle_USB2.0_8P, J3 Conn_01x02_Socket, J4 Conn_01x02_Socket, J5 Conn_01x03_Socket, Q1 PMOS, Q2 2N7002K, Q3 PMOS, Q4 PMOS, U1 AP2112K-3.3, U2 ESP32-WROOM-32-N8R2, U3 INMP441, U4 MAX98357A, U5 MAX98357A, U6 TP4056, U7 MAX98357AETE+T, U8 MAX98357AETE+T

Commit message: refactor(hardware): split KiCad and printed-part trees; add Echoes V2
Other:
- board text added: "Marajoara V3"
- board text removed: "Marajoara V2"
Changed lines of the file:
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@@
 		)
 	)
-	(gr_text "Marajoara V2"
+	(gr_text "Marajoara V3"
 		(at 241.215708 57.2707 0)
 		(layer "F.SilkS")
