File: Hardware/PCBs/Marajoara_V3/Marajoara_V3.kicad_sch (KiCad schematic)
At the start: 122 parts, among them J1 Conn_01x02_Socket, J2 USB_C_Receptacle_USB2.0_8P, J3 Conn_01x02_Socket, J4 Conn_01x02_Socket, J5 Conn_01x03_Socket, Q1 PMOS, Q2 2N7002K, Q3 PMOS, Q4 PMOS, U1 AP2112K-3.3, U2 ESP32-WROOM-32-N8R2, U3 INMP441, U4 MAX98357A, U5 MAX98357A, U6 TP4056, U7 MAX98357AETE+T, U8 MAX98357AETE+T

Commit message: refactor(hardware): split KiCad and printed-part trees; add Echoes V2
Parts:
- added R35, R37: 100k, Resistor_SMD:R_0805_2012Metric_Pad1.20x1.40mm_HandSolder, symbol Device:R
Connections:
- net +3.3V: now also R35.2, R37.2
- net SD_D1: no longer U2.26 (IO4)
- net VCC: no longer R20.2
- net V_REG: now also R20.2
- net CHRG: now reaches D4.1 (K), U6.7 (CHRG#)
- net CHRG: now also U2.26 (IO4)
- net STDBY: now reaches U2.7 (IO35)
- net STDBY: now also D3.1 (K), U6.6 (STDBY#), R35.1, R37.1
Other:
- moved on the sheet: R7, R8
